File: starbie-kicad/starbie-kicad.kicad_sch (KiCad schematic)
At the start: 0 parts

Commit message: drawn scematics for starbie
on KiCAD
Parts:
- added J1: Conn_01x04_Pin, Imported Parts:Display_128x64_096_I2C, symbol Connector:Conn_01x04_Pin
- added J2: Conn_01x08_Pin, Connector_PinHeader_2.54mm:PinHeader_1x08_P2.54mm_Vertical, symbol Connector:Conn_01x08_Pin
- added R1: R, Resistor_THT:R_Axial_DIN0204_L3.6mm_D1.6mm_P7.62mm_Horizontal, symbol Device:R
- added SW1, SW2: SW_Push, Button_Switch_Keyboard:SW_Cherry_MX_1.00u_PCB, symbol Switch:SW_Push
- added U1: XIAO-ESP32-C3-SMD, Sensor:Aosong_DHT11_5.5x12.0_P2.54mm, symbol Seeed_Studio_XIAO_Series:XIAO-ESP32-C3-SMD
- added U2: DHT11, Imported Parts:XIAO-ESP32-C6-DIP, symbol Sensor:DHT11
Connections:
- new net +3.3V: J1.2 (Pin_2), J2.1 (Pin_1), R1.1, U1.12 (3V3_OUT), U2.1 (VDD)
- new net +5V: U1.14 (VBUS)
- new net DHT11 DATA: R1.2, U1.2 (D1), U2.2 (DATA)
- new net GND: J1.1 (Pin_1), J2.2 (Pin_2), SW1.2, SW2.2, U1.13 (GND), U1.18 (GND), U2.4 (GND)
- new net GPIO2: SW1.1, U1.3 (D2)
- new net GPIO3: SW2.1, U1.4 (D3)
- new net SCL: J1.3 (Pin_3), J2.3 (Pin_3), U1.5 (D4)
- new net SDA: J1.4 (Pin_4), J2.4 (Pin_4), U1.6 (D5)
- no-connect marks 0 -> 17
